Commit message: update dynamics

File: tutorial_gazebo/urdf/forktruck_body.urdf.xacro (robot description, xacro)
@@ -124,6 +124,9 @@
     </collision>
   </link>
-  <joint name="vplate_joint" type="fixed">
+  <joint name="vplate_joint" type="prismatic">
     <origin xyz=".10 -0.0 0.04" rpy="0 0 0"/>
+    <axis xyz="1 0 0" />
+    <limit effort="2000.0" lower="0" upper="0.6" velocity="0.2"/>
+    <dynamics damping="1000.0"/>
     <parent link="base_link"/>
     <child link="vplate"/>
@@ -202,12 +205,71 @@
     </collision>
   </link>
-  <joint name="fork_joint" type="fixed">
-    <origin xyz="0.0 0.0 -0.35" rpy="0 0 0"/>
+  <joint name="fork_joint" type="prismatic">
+    <origin xyz="0.0 0.0 -0.5" rpy="0 0 0"/>
     <axis xyz="0 0 1" />
-    <limit effort="10.0" lower="-0.35" upper="3.5" velocity="0.2"/>
+    <limit effort="2000.0" lower="0.0" upper="2.7" velocity="0.2"/>
     <dynamics damping="1000.0"/>
     <parent link="vplate"/>
     <child link="fork"/>
   </joint>
+<link name="ltooth">
+    <inertial>
+      <origin xyz="0 0 0"/>
+      <mass value="5" />
+      <inertia ixx="0.021" ixy="0.0" ixz="0.0"
+        iyy="0.021" iyz="0.0" izz="0.021" />
+    </inertial>
+    <visual>
+      <origin xyz="0 0 0.0"  rpy="${0.5*M_PI} ${0.0*M_PI} ${0.5*M_PI}" />
+      <geometry>
+        <mesh filename="package://tutorial_gazebo/meshes/folktruck_forktooth.stl" scale="${ratio} ${ratio} ${ratio}"/>
+      </geometry>
+      <material name="orange" />
+    </visual>
+    <collision>
+      <origin xyz="0 0 0.0"  rpy="${0.5*M_PI} ${0.0*M_PI} ${0.5*M_PI}" />
+      <geometry>
+        <mesh filename="package://tutorial_gazebo/meshes/folktruck_forktooth.stl" scale="${ratio} ${ratio} ${ratio}"/>
+      </geometry>
+    </collision>
+  </link>
+  <joint name="ltooth_joint" type="prismatic">
+    <origin xyz="0.0 0.0 0.0" rpy="0 0 0"/>
+    <axis xyz="0 -1 0" />
+    <limit effort="500.0" lower="0.0" upper="0.5" velocity="0.2"/>
+    <dynamics damping="1000.0"/>
+    <parent link="fork"/>
+    <child link="ltooth"/>
+  </joint>
+<link name="rtooth">
+    <inertial>
+      <origin xyz="0 0 0"/>
+      <mass value="5" />
+      <inertia ixx="0.021" ixy="0.0" ixz="0.0"
+        iyy="0.021" iyz="0.0" izz="0.021" />
+    </inertial>
+    <visual>
+      <origin xyz="0 0 0.0"  rpy="${0.5*M_PI} ${0.0*M_PI} ${0.5*M_PI}" />
+      <geometry>
+        <mesh filename="package://tutorial_gazebo/meshes/folktruck_forktooth.stl" scale="${ratio} ${ratio} ${ratio}"/>
+      </geometry>
+      <material name="orange" />
+    </visual>
+    <collision>
+      <origin xyz="0 0 0.0"  rpy="${0.5*M_PI} ${0.0*M_PI} ${0.5*M_PI}" />
+      <geometry>
+        <mesh filename="package://tutorial_gazebo/meshes/folktruck_forktooth.stl" scale="${ratio} ${ratio} ${ratio}"/>
+      </geometry>
+    </collision>
+  </link>
+  <joint name="rtooth_joint" type="prismatic">
+    <origin xyz="0.0 -1.45 0.0" rpy="0 0 0"/>
+    <axis xyz="0 1 0" />
+    <limit effort="500.0" lower="0.0" upper="0.5" velocity="0.2"/>
+    <dynamics damping="1000.0"/>
+    <parent link="fork"/>
+    <child link="rtooth"/>
+    <mimic joint="ltooth_joint" multiplier="1" offset="0"/>
+  </joint>
 <link name="plate">
     <inertial>
@@ -220,5 +282,5 @@
       <origin xyz="0 0 0.0" rpy="0 0 0"/>
       <geometry>
-        <box size="0.2 0.2 0.012" />
+        <box size="1.8 0.12 0.02" />
       </geometry>
       <material name="orange" />
@@ -232,6 +294,6 @@
   </link>
   <joint name="plate_joint" type="fixed">
-    <origin xyz="0.0 0 0.12" rpy="0 0 0"/>
-    <parent link="base_link"/>
+    <origin xyz="-0.45 0 -0.25" rpy="0 0 0"/>
+    <parent link="vplate"/>
     <child link="plate"/>
   </joint>
@@ -305,5 +367,13 @@
     <child link="laser" />
   </joint>
-  <!--transmission name="tran1">
+  <transmission name="tran0">
+    <type>transmission_interface/SimpleTransmission</type>
+    <joint name="vplate_joint"/>
+    <actuator name="motor0">
+      <hardwareInterface>EffortJointInterface</hardwareInterface>
+      <mechanicalReduction>1</mechanicalReduction>
+    </actuator>
+  </transmission>
+  <transmission name="tran1">
     <type>transmission_interface/SimpleTransmission</type>
     <joint name="fork_joint"/>
@@ -312,5 +382,21 @@
       <mechanicalReduction>1</mechanicalReduction>
     </actuator>
-  </transmission-->
+  </transmission>
+  <transmission name="tran2">
+    <type>transmission_interface/SimpleTransmission</type>
+    <joint name="ltooth_joint"/>
+    <actuator name="motor2">
+      <hardwareInterface>EffortJointInterface</hardwareInterface>
+      <mechanicalReduction>1</mechanicalReduction>
+    </actuator>
+  </transmission>
+  <transmission name="tran3">
+    <type>transmission_interface/SimpleTransmission</type>
+    <joint name="rtooth_joint"/>
+    <actuator name="motor3">
+      <hardwareInterface>EffortJointInterface</hardwareInterface>
+      <mechanicalReduction>1</mechanicalReduction>
+    </actuator>
+  </transmission>
 <!--Painting color for all the joints-->
   <gazebo reference="f_wheel_link">
@@ -344,4 +430,14 @@
    <material>Gazebo/FlatBlack</material>
   </gazebo>
+  <gazebo reference="ltooth">
+    <mu1>100.2</mu1>
+    <mu2>100.2</mu2>
+   <material>Gazebo/Green</material>
+  </gazebo>
+  <gazebo reference="rtooth">
+    <mu1>100.2</mu1>
+    <mu2>100.2</mu2>
+   <material>Gazebo/Red</material>
+  </gazebo>
   </xacro:macro>
 </robot>

File: tutorial_gazebo/urdf/forktruck_plugin.xacro (robot description, xacro)
@@ -1,4 +1,9 @@
 <?xml version="1.0"?>
 <robot>
+	<gazebo>
+	  <plugin name="gazebo_ros_control" filename="libgazebo_ros_control.so">
+		  <robotParam>/robot_description</robotParam>
+	  </plugin>
+	</gazebo>
 <!--gazebo reference="laser">
     <sensor type="gpu_ray" name="head_hokuyo_sensor">

Commit message: ameliorate mesh files

File: tutorial_gazebo/urdf/forktruck_body.urdf.xacro (robot description, xacro)
@@ -26,8 +26,8 @@
   <link name="base_link">
     <inertial>
-      <mass value="80" />
+      <mass value="800" />
       <origin xyz="0 0 0" />
-      <inertia ixx="0.01" ixy="0.0" ixz="0.0"
-        iyy="0.01" iyz="0.0" izz="0.5" />
+      <inertia ixx="11" ixy="0.0" ixz="0.0"
+        iyy="10" iyz="0.0" izz="15" />
     </inertial>
     <visual>
@@ -52,7 +52,7 @@
     <inertial>
       <origin xyz="0 0 0"/>
-      <mass value="10.01" />
-      <inertia ixx="0.001" ixy="0.0" ixz="0.0"
-        iyy="0.001" iyz="0.0" izz="0.001" />
+      <mass value="200" />
+      <inertia ixx="5.01" ixy="0.0" ixz="0.0"
+        iyy="2.1" iyz="0.0" izz="4.1" />
     </inertial>
     <visual>
@@ -79,7 +79,7 @@
     <inertial>
       <origin xyz="0 0 0"/>
-      <mass value="20" />
-      <inertia ixx="0.001" ixy="0.0" ixz="0.0"
-        iyy="0.001" iyz="0.0" izz="0.001" />
+      <mass value="200" />
+      <inertia ixx="5.01" ixy="0.0" ixz="0.0"
+        iyy="2.1" iyz="0.0" izz="4.1" />
     </inertial>
     <visual>
@@ -128,5 +128,5 @@
     <axis xyz="1 0 0" />
     <limit effort="2000.0" lower="0" upper="0.6" velocity="0.2"/>
-    <dynamics damping="1000.0"/>
+    <dynamics damping="1.0"/>
     <parent link="base_link"/>
     <child link="vplate"/>
@@ -180,5 +180,5 @@
   </link>
   <joint name="rcynldr_joint" type="fixed">
-        <origin xyz="0.4 -0.53 1.55" rpy="0 0 0"/>
+    <origin xyz="0.4 -0.53 1.55" rpy="0 0 0"/>
     <parent link="vplate"/>
     <child link="rcynldr"/>
@@ -208,6 +208,6 @@
     <origin xyz="0.0 0.0 -0.5" rpy="0 0 0"/>
     <axis xyz="0 0 1" />
-    <limit effort="2000.0" lower="0.0" upper="2.7" velocity="0.2"/>
-    <dynamics damping="1000.0"/>
+    <limit effort="5000.0" lower="0.0" upper="2.7" velocity="0.2"/>
+    <dynamics damping="1.0"/>
     <parent link="vplate"/>
     <child link="fork"/>
@@ -238,5 +238,5 @@
     <axis xyz="0 -1 0" />
     <limit effort="500.0" lower="0.0" upper="0.5" velocity="0.2"/>
-    <dynamics damping="1000.0"/>
+    <dynamics damping="1.0"/>
     <parent link="fork"/>
     <child link="ltooth"/>
@@ -267,5 +267,5 @@
     <axis xyz="0 1 0" />
     <limit effort="500.0" lower="0.0" upper="0.5" velocity="0.2"/>
-    <dynamics damping="1000.0"/>
+    <dynamics damping="1.0"/>
     <parent link="fork"/>
     <child link="rtooth"/>
@@ -431,11 +431,23 @@
   </gazebo>
   <gazebo reference="ltooth">
-    <mu1>100.2</mu1>
-    <mu2>100.2</mu2>
+    <kp>1000000.0</kp>
+    <kd>1</kd>
+    <mu1>10000000.0</mu1>
+    <mu2>10000000.0</mu2>
+    <fdir1>1 1 0</fdir1>
+    <maxVel>1.0</maxVel>
+    <maxContacts>100</maxContacts>
+    <minDepth>0.00</minDepth>
    <material>Gazebo/Green</material>
   </gazebo>
   <gazebo reference="rtooth">
-    <mu1>100.2</mu1>
-    <mu2>100.2</mu2>
+    <kp>1000000.0</kp>
+    <kd>1.0</kd>
+    <mu1>10000000.0</mu1>
+    <mu2>10000000.0</mu2>
+    <fdir1>1 1 0</fdir1>
+    <maxVel>1.0</maxVel>
+    <minDepth>0.00</minDepth>
+    <maxContacts>100</maxContacts>
    <material>Gazebo/Red</material>
   </gazebo>
