Commit message: add new factory

File: tutorial_gazebo/urdf/forktruck_body_nojoint.urdf.xacro (robot description, xacro)
@@ -149,5 +149,5 @@
     </collision>
   </link>
-  <joint name="vplate_joint" type="prismatic">
+  <joint name="vplate_joint" type="fixed">
     <origin xyz=".10 -0.0 0.04" rpy="0 0 0"/>
     <axis xyz="1 0 0" />
@@ -230,5 +230,5 @@
     </collision>
   </link>
-  <joint name="fork_joint" type="prismatic">
+  <joint name="fork_joint" type="fixed">
     <origin xyz="0.0 0.0 -0.5" rpy="0 0 0"/>
     <axis xyz="0 0 1" />
@@ -259,5 +259,5 @@
     </collision>
   </link>
-  <joint name="ltooth_joint" type="prismatic">
+  <joint name="ltooth_joint" type="fixed">
     <origin xyz="0.0 0.0 0.0" rpy="0 0 0"/>
     <axis xyz="0 -1 0" />
@@ -288,5 +288,5 @@
     </collision>
   </link>
-  <joint name="rtooth_joint" type="prismatic">
+  <joint name="rtooth_joint" type="fixed">
     <origin xyz="0.0 -1.45 0.0" rpy="0 0 0"/>
     <axis xyz="0 1 0" />
@@ -370,5 +370,5 @@
     </inertial>
   </link>
-  <joint name="camera_joint" type="prismatic">
+  <joint name="camera_joint" type="fixed">
     <origin xyz="0.0 0.0 -0.0" rpy="0 0 0"/>
     <axis xyz="0 0 1" />

File: tutorial_gazebo/urdf/forktruck_plugin.xacro (robot description, xacro)
@@ -6,8 +6,8 @@
 	  </plugin>
 	</gazebo>
-<!--gazebo reference="laser">
+<gazebo reference="laser">
     <sensor type="gpu_ray" name="head_hokuyo_sensor">
       <pose>0 0 0 0 0 0</pose>
-      <visualize>false</visualize>
+      <visualize>true</visualize>
       <update_rate>40</update_rate>
       <ray>
@@ -36,4 +36,41 @@
       </plugin>
     </sensor>
+  </gazebo>
+  <!--gazebo reference="camera_link">
+    <sensor type="depth" name="kinect_frame_sensor" >
+      <pose>0 0 0 0 1.57079632679 0</pose>
+      <always_on>true</always_on>
+      <update_rate>10</update_rate>
+      <camera>
+        <horizontal_fov>0.994837673637</horizontal_fov>
+        <image>
+          <format>R8G8B8</format>
+          <width>640</width>
+          <height>480</height>
+        </image>
+        <clip>
+          <near>0.01</near>
+          <far>50</far>
+        </clip>
+      </camera>
+      <plugin filename="libgazebo_ros_openni_kinect.so" name="kinect_controller">
+        <alwaysOn>true</alwaysOn>
+        <updateRate>10</updateRate>
+        <cameraName>kinect</cameraName>
+        <imageTopicName>/kinect/ir/image_raw</imageTopicName>
+        <cameraInfoTopicName>/kinect/ir/camera_info</cameraInfoTopicName>
+        <depthImageTopicName>/kinect/depth/image_raw</depthImageTopicName>
+        <depthCameraInfoTopicName>/kinect/camera_info</depthCameraInfoTopicName>
+        <depthImageCameraInfoTopicName>/kinect/depth/camera_info</depthImageCameraInfoTopicName>
+        <pointCloudTopicName>/kinect/depth/points</pointCloudTopicName>
+        <pointCloudCutoff>0.5</pointCloudCutoff>
+        <frameName>kinect_image_frame</frameName>
+        <distortionK1>0.0001</distortionK1>
+        <distortionK2>0.001</distortionK2>
+        <distortionK3>0.0001</distortionK3>
+        <distortionT1>0.0001</distortionT1>
+        <distortionT2>0.001</distortionT2>
+      </plugin>
+    </sensor>
   </gazebo-->
   <gazebo>
